File: Pi1551-III Module Panel/Pi1551-III Module Panel.kicad_pcb (KiCad board)
At the start: 2 copper layers, 100 x 23.2 mm, 15 parts, among them IC1 OLED, J1 Module Panel, M1 Mounting_Pin, M2 Mounting_Pin, M3 Mounting_Pin, M4 Mounting_Pin, SW1 BACK, SW2 INSERT

Commit message: rebranding to Pi1551-III
Other:
- board text added: "BulkyMIDI-32 Pi1551-III Panel (rev. A) github.com/tebl"
- board text removed: "BulkyMIDI-32 Pi1541-III Panel (rev. A) github.com/tebl"
Changed lines of the file:
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@@
     (effects (font (size 0.8 0.8) (thickness 0.1)) (justify mirror))
   )
-  (gr_text "BulkyMIDI-32\nPi1541-III Panel (rev. A)\ngithub.com/tebl" (at 94.1 122.849 270) (layer B.SilkS)
+  (gr_text "BulkyMIDI-32\nPi1551-III Panel (rev. A)\ngithub.com/tebl" (at 94.1 122.849 270) (layer B.SilkS)
     (effects (font (size 0.8 0.8) (thickness 0.1)) (justify mirror))
   )
