File: faceplates/Pi1551-III Module FP1/Pi1551-III Module FP1.kicad_pcb (KiCad board)
At the start: 2 copper layers, 100 x 35 mm, 9 parts, among them M1 Mounting_Pin, M2 Mounting_Pin, M3 Mounting_Pin, M4 Mounting_Pin

Commit message: upgrade to KiCad 9.0.7
Other:
- net class Default removed
- net class PWR removed
- board text added: "Module FP1 (rev. A)"
- board text removed: "BulkyMIDI-32 Module FP2 (rev. B) github.com/tebl"
